Commit message: minor robot model fixes

File: src/jetbot/description/gazebo_control.xacro (robot description, xacro)
@@ -6,5 +6,5 @@
             <left_joint>left_wheel_joint</left_joint>
             <right_joint>right_wheel_joint</right_joint>
-            <wheel_separation>0.27</wheel_separation>
+            <wheel_separation>0.522</wheel_separation>
             <wheel_diameter>0.06</wheel_diameter>
             <!-- Limits -->

File: src/jetbot/description/lidar.xacro (robot description, xacro)
@@ -34,5 +34,5 @@
         <sensor name="laser" type="ray">
             <pose> 0 0 0 0 0 0 </pose>
-            <visualize>true</visualize>
+            <visualize>0</visualize>
             <update_rate>10</update_rate>
             <ray>

File: src/jetbot/description/robot_core.xacro (robot description, xacro)
@@ -109,5 +109,5 @@
         <parent link="chassis" />
         <child link="caster_wheel_front" />
-        <origin xyz="${caster_wheel_offset_x} 0 ${caster_wheel_offset_z}" />
+        <origin xyz="${caster_wheel_offset_x} 0 ${caster_wheel_offset_z+0.001}" />
     </joint>
     <link name="caster_wheel_front">
@@ -135,5 +135,5 @@
         <parent link="chassis" />
         <child link="caster_wheel_back" />
-        <origin xyz="${-caster_wheel_offset_x} 0 ${caster_wheel_offset_z}" />
+        <origin xyz="${-caster_wheel_offset_x} 0 ${caster_wheel_offset_z+0.001}" />
     </joint>
     <link name="caster_wheel_back">
