Commit message: redo of robot geometry added second castor wheel for stability fixed mass not being taken from params move/resize lidar and camera change chassis from box to cylinder decrase wheel acceleration

File: src/jetbot/description/camera.xacro (robot description, xacro)
@@ -1,8 +1,9 @@
 <?xml version="1.0"?>
 <robot xmlns:xacro="http://www.ros.org/wiki/xacro">
+    <xacro:include filename="dimensions.xacro" />
     <joint name="camera_joint" type="fixed">
         <parent link="chassis" />
         <child link="camera_link" />
-        <origin xyz="0.276 0 0.181" rpy="0 0.18 0" />
+        <origin xyz="${chassis_radius - 0.01} 0 ${chassis_length + 0.03}" rpy="0 0.1 0" />
     </joint>
     <link name="camera_link">
@@ -14,7 +15,7 @@
         </visual>
         <visual>
-            <origin xyz="0 0 -0.05" />
+            <origin xyz="0 0 -0.015" />
             <geometry>
-                <cylinder radius="0.002" length="0.1" />
+                <cylinder radius="0.002" length="0.03" />
             </geometry>
             <material name="black" />

File: src/jetbot/description/gazebo_control.xacro (robot description, xacro)
@@ -6,9 +6,9 @@
             <left_joint>left_wheel_joint</left_joint>
             <right_joint>right_wheel_joint</right_joint>
-            <wheel_separation>0.297</wheel_separation>
-            <wheel_diameter>0.066</wheel_diameter>
+            <wheel_separation>0.27</wheel_separation>
+            <wheel_diameter>0.06</wheel_diameter>
             <!-- Limits -->
             <max_wheel_torque>200</max_wheel_torque>
-            <max_wheel_acceleration>10.0</max_wheel_acceleration>
+            <max_wheel_acceleration>2.5</max_wheel_acceleration>
             <!-- Output -->
             <odometry_frame>odom</odometry_frame>

File: src/jetbot/description/lidar.xacro (robot description, xacro)
@@ -1,8 +1,9 @@
 <?xml version="1.0"?>
 <robot xmlns:xacro="http://www.ros.org/wiki/xacro">
+    <xacro:include filename="dimensions.xacro" />
     <joint name="laser_joint" type="fixed">
         <parent link="chassis" />
         <child link="laser_frame" />
-        <origin xyz="0.122 0 0.212" rpy="0 0 0" />
+        <origin xyz="0 0 ${chassis_length + 0.08}" rpy="0 0 0" />
     </joint>
     <link name="laser_frame">
@@ -16,5 +17,5 @@
             <origin xyz="0 0 -0.05" />
             <geometry>
-                <cylinder radius="0.01" length="0.1" />
+                <cylinder radius="0.01" length="0.06" />
             </geometry>
             <material name="black" />

File: src/jetbot/description/robot_core.xacro (robot description, xacro)
@@ -2,19 +2,5 @@
 <robot xmlns:xacro="http://www.ros.org/wiki/xacro">
     <xacro:include filename="inertial_macros.xacro" />
-    <xacro:property name="chassis_length" value="0.335" />
-    <xacro:property name="chassis_width" value="0.265" />
-    <xacro:property name="chassis_height" value="0.138" />
-    <xacro:property name="chassis_mass" value="1.0" />
-    <xacro:property name="wheel_radius" value="0.033" />
-    <xacro:property name="wheel_thickness" value="0.026" />
-    <xacro:property name="wheel_mass" value="0.05" />
-    <xacro:property name="wheel_offset_x" value="0.226" />
-    <xacro:property name="wheel_offset_y" value="0.1485" />
-    <xacro:property name="wheel_offset_z" value="0.01" />
-    <xacro:property name="caster_wheel_radius" value="0.01" />
-    <xacro:property name="caster_wheel_mass" value="0.01" />
-    <xacro:property name="caster_wheel_offset_x" value="0.075" />
-    <xacro:property name="caster_wheel_offset_z"
-        value="${wheel_offset_z - wheel_radius + caster_wheel_radius}" />
+    <xacro:include filename="dimensions.xacro" />
     <material name="white">
         <color rgba="1 1 1 1" />
@@ -33,6 +19,5 @@
     </material>
     <!-- BASE LINK -->
-    <link name="base_link">
-    </link>
+    <link name="base_link" />
     <!-- BASE_FOOTPRINT LINK -->
     <joint name="base_footprint_joint" type="fixed">
@@ -41,30 +26,28 @@
         <origin xyz="0 0 0" rpy="0 0 0" />
     </joint>
-    <link name="base_footprint">
-    </link>
+    <link name="base_footprint"/>
     <!-- CHASSIS LINK -->
     <joint name="chassis_joint" type="fixed">
         <parent link="base_link" />
         <child link="chassis" />
-        <origin xyz="${-wheel_offset_x} 0 ${-wheel_offset_z}" />
+        <origin xyz="0 0 ${-wheel_offset_z}" />
     </joint>
     <link name="chassis">
         <visual>
-            <origin xyz="${chassis_length/2} 0 ${chassis_height/2}" />
+            <origin xyz="0 0 ${chassis_length/2}" />
             <geometry>
-                <box size="${chassis_length} ${chassis_width} ${chassis_height}" />
+                <cylinder radius="${chassis_radius}" length="${chassis_length}" />
             </geometry>
             <material name="grey" />
         </visual>
         <collision>
-            <origin xyz="${chassis_length/2} 0 ${chassis_height/2}" />
+            <origin xyz="0 0 ${chassis_length/2}" />
             <geometry>
-                <box size="${chassis_length} ${chassis_width} ${chassis_height}" />
+                <cylinder radius="${chassis_radius}" length="${chassis_length}" />
             </geometry>
         </collision>
-        <xacro:inertial_box mass="0.5" x="${chassis_length}" y="${chassis_width}"
-            z="${chassis_height}">
-            <origin xyz="${chassis_length/2} 0 ${chassis_height/2}" rpy="0 0 0" />
-        </xacro:inertial_box>
+        <xacro:inertial_cylinder mass="${chassis_mass}" length="${chassis_length}" radius="${chassis_radius}">
+            <origin xyz="0 0 ${chassis_length/2}" rpy="0 0 0" />
+        </xacro:inertial_cylinder>
     </link>
     <!-- LEFT WHEEL LINK -->
@@ -122,11 +105,11 @@
         <material>Gazebo/Blue</material>
     </gazebo>
-    <!-- CASTER WHEEL LINK -->
-    <joint name="caster_wheel_joint" type="fixed">
+    <!-- CASTER WHEEL LINKS -->
+    <joint name="caster_front_joint" type="fixed">
         <parent link="chassis" />
-        <child link="caster_wheel" />
+        <child link="caster_wheel_front" />
         <origin xyz="${caster_wheel_offset_x} 0 ${caster_wheel_offset_z}" />
     </joint>
-    <link name="caster_wheel">
+    <link name="caster_wheel_front">
         <visual>
             <geometry>
@@ -144,5 +127,31 @@
         </xacro:inertial_sphere>
     </link>
-    <gazebo reference="caster_wheel">
+    <gazebo reference="caster_wheel_front">
+        <material>Gazebo/White</material>
+        <mu1 value="0" />
+        <mu2 value="0" />
+    </gazebo>
+    <joint name="caster_back_joint" type="fixed">
+        <parent link="chassis" />
+        <child link="caster_wheel_back" />
+        <origin xyz="${-caster_wheel_offset_x} 0 ${caster_wheel_offset_z}" />
+    </joint>
+    <link name="caster_wheel_back">
+        <visual>
+            <geometry>
+                <sphere radius="${caster_wheel_radius}" />
+            </geometry>
+            <material name="white" />
+        </visual>
+        <collision>
+            <geometry>
+                <sphere radius="${caster_wheel_radius}" />
+            </geometry>
+        </collision>
+        <xacro:inertial_sphere mass="${caster_wheel_mass}" radius="${caster_wheel_radius}">
+            <origin xyz="0 0 0" rpy="0 0 0" />
+        </xacro:inertial_sphere>
+    </link>
+    <gazebo reference="caster_wheel_back">
         <material>Gazebo/White</material>
         <mu1 value="0" />

Commit message: optimizations and cleanup

File: src/jetbot/description/camera.xacro (robot description, xacro)
@@ -44,9 +44,4 @@
                 <frameName>camera_link</frameName>
                 <hackBaseline>0.07</hackBaseline>
-                <distortionK1>0.0</distortionK1>
-                <distortionK2>0.0</distortionK2>
-                <distortionK3>0.0</distortionK3>
-                <distortionT1>0.0</distortionT1>
-                <distortionT2>0.0</distortionT2>
               </plugin>
             <always_on>1</always_on>

File: src/jetbot/description/dimensions.xacro (robot description, xacro)
@@ -2,5 +2,5 @@
 <robot xmlns:xacro="http://www.ros.org/wiki/xacro">
     <xacro:property name="chassis_length" value="0.10" />
-    <xacro:property name="chassis_radius" value="0.25" />
+    <xacro:property name="chassis_radius" value="0.15" />
     <xacro:property name="chassis_mass" value="1.0" />
     <xacro:property name="wheel_radius" value="0.03" />
